File: schematic/workshop_piano.kicad_pcb (KiCad board)
At the start: 2 copper layers, 102 x 34 mm, 37 parts, among them J1 Jack-DC, J2 Conn_01x05_Pin, J3 AudioJack3, SW1 SW_SPST, SW2 SW_SPST, SW3 SW_SPST, SW4 SW_SPST, SW5 SW_SPST, SW6 SW_SPST, SW7 SW_SPST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

Commit message: 回路図の修正をAWに反映
Parts:
- C1: value C_Polarized -> 10u
- renumbered J2 to J1, J1 to J2
Connections:
- R14 pad 1: Net-(U1-PWM1/CWG1A/T0CKI/RC5) -> /LED6
- U1 pad 2: AUDIO_OUTPUT -> /LED6
- U1 pad 5: Net-(U1-PWM1/CWG1A/T0CKI/RC5) -> AUDIO_OUTPUT
Routing:
- net /LED6: track 0.00 -> 34.3 mm, vias 0 -> 2
- net Net-(U1-PWM1/CWG1A/T0CKI/RC5): track 26.6 -> 0.00 mm, vias 1 -> 0
- net AUDIO_OUTPUT: track 42.8 -> 35.1 mm
- net Net-(C1-Pad2): track 19.7 -> 18.9 mm
